File: HW2 Files/CircuitSchematic.brd (EAGLE design)
At the start: 50 x 50 mm, 23 parts

Commit message: Added missing connections
To do:
- Add pictures
- Add name and info
Routing:
- net +3V3: track 105.7 -> 169.9 mm, vias 0 -> 3
- net A4/LED: track 83.4 -> 84.9 mm
Changed lines of the file:
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@@
 <wire x1="29.21" y1="46.99" x2="29.21" y2="41.91" width="0.4064" layer="1"/>
 <wire x1="29.21" y1="46.99" x2="33.02" y2="46.99" width="0.4064" layer="16"/>
-<wire x1="29.21" y1="41.91" x2="25.4" y2="38.1" width="0.4064" layer="1"/>
+<wire x1="25.4" y1="38.1" x2="29.21" y2="41.91" width="0.4064" layer="1"/>
 <wire x1="25.4" y1="33.02" x2="25.4" y2="38.1" width="0.4064" layer="1"/>
 <wire x1="25.4" y1="33.02" x2="25.4" y2="15.24" width="0.4064" layer="1"/>
@@
 <wire x1="16.51" y1="15.24" x2="12.065" y2="19.685" width="0.4064" layer="1"/>
 <wire x1="7.62" y1="9.525" x2="1.905" y2="9.525" width="0.4064" layer="16"/>
-<wire x1="1.905" y1="9.525" x2="1.27" y2="10.16" width="0.4064" layer="16"/>
-<wire x1="7.62" y1="9.525" x2="16.51" y2="12.7" width="0" layer="19" extent="16-16"/>
-<wire x1="1.27" y1="19.05" x2="1.27" y2="10.16" width="0" layer="19" extent="1-1"/>
+<wire x1="1.27" y1="10.16" x2="1.905" y2="9.525" width="0.4064" layer="16"/>
+<wire x1="7.62" y1="34.091975" x2="7.62" y2="38.1" width="0.4064" layer="1"/>
+<wire x1="6.862" y1="33.333975" x2="7.62" y2="34.091975" width="0.4064" layer="1"/>
+<wire x1="6.862" y1="24.642" x2="1.27" y2="19.05" width="0.4064" layer="1"/>
+<wire x1="6.862" y1="24.642" x2="6.862" y2="33.333975" width="0.4064" layer="1"/>
+<via x="7.62" y="38.1" extent="1-16" drill="0.5"/>
+<wire x1="7.62" y1="38.1" x2="25.4" y2="38.1" width="0.4064" layer="16"/>
+<via x="25.4" y="38.1" extent="1-16" drill="0.5"/>
+<wire x1="10.918" y1="8.576025" x2="10.473975" y2="8.132" width="0.4064" layer="1"/>
+<wire x1="9.402" y1="8.132" x2="7.62" y2="6.35" width="0.4064" layer="1"/>
+<wire x1="10.473975" y1="8.132" x2="9.402" y2="8.132" width="0.4064" layer="1"/>
+<wire x1="21.59" y1="11.43" x2="12.53315625" y2="11.43" width="0.4064" layer="1"/>
+<wire x1="12.53315625" y1="11.43" x2="10.918" y2="9.81484375" width="0.4064" layer="1"/>
+<wire x1="10.918" y1="9.81484375" x2="10.918" y2="8.576025" width="0.4064" layer="1"/>
+<via x="7.62" y="6.35" extent="1-16" drill="0.5"/>
+<wire x1="7.62" y1="6.35" x2="5.08" y2="6.35" width="0.4064" layer="16"/>
+<wire x1="5.08" y1="6.35" x2="1.27" y2="10.16" width="0.4064" layer="16"/>
 </signal>
 <signal name="MCLR">
@@
 <wire x1="5.08" y1="41.91" x2="5.08" y2="25.4" width="0.4064" layer="1"/>
 <wire x1="5.08" y1="25.4" x2="1.27" y2="21.59" width="0.4064" layer="1"/>
+<wire x1="24.13" y1="3.81" x2="25.654" y2="3.81" width="0.4064" layer="16"/>
 </signal>
 <signal name="B4/USER">
@@
 </signal>
 </signals>
+<errors>
+</errors>
 </board>
 </drawing>
